Commit message: gazebo simulation edits

File: baxter_description/urdf/baxter.urdf.xacro (robot description, xacro)
@@ -1,15 +1,15 @@
 <?xml version="1.0" ?>
 <robot name="baxter" xmlns:xacro="http://www.ros.org/wiki/xacro">
-  <xacro:arg name="gazebo" default="false"/>
+  <xacro:arg name="gazebo" default="true"/>
   <xacro:arg name="pedestal" default="true"/>
   <xacro:property name="PI" value="3.1415927"/>
   <!-- Baxter Base URDF -->
   <xacro:include filename="$(find baxter_description)/urdf/baxter_base/baxter_base.urdf.xacro">
-<!--     <xacro:arg name="gazebo" value="$(arg gazebo)"/> -->
+     <xacro:arg name="gazebo" value="$(arg gazebo)"/>
   </xacro:include>
   <!-- Baxter Pedestal -->
   <xacro:if value="$(arg pedestal)">
     <xacro:include filename="$(find baxter_description)/urdf/pedestal/pedestal.xacro">
-<!--       <xacro:arg name="gazebo" value="$(arg gazebo)"/> -->
+       <xacro:arg name="gazebo" value="$(arg gazebo)"/>
     </xacro:include>
   </xacro:if>
@@ -19,4 +19,4 @@
   <xacro:include filename="$(find baxter_description)/urdf/right_end_effector.urdf.xacro" />
   <!-- Gazebo plugins -->
-  <xacro:include filename="$(find baxter_description)/urdf/gazebosim.urdf.xacro" />
+  <!--xacro:include filename="$(find baxter_description)/urdf/gazebosim.urdf.xacro" /-->
 </robot>

File: baxter_description/urdf/baxter_base/baxter_base.gazebo.xacro (robot description, xacro)
@@ -1,17 +1,11 @@
 <?xml version="1.0" ?>
 <robot name="baxter" xmlns:xacro="http://www.ros.org/wiki/xacro">
-  <!-- ros_control plugin -->
-  <gazebo>
-    <plugin name="baxter_ros_control" filename="libbaxter_gazebo_ros_control.so">
-      <robotNamespace>/robot</robotNamespace>
-    </plugin>
-  </gazebo>
   <!-- Gazebo-Specific Link Properties -->
   <gazebo reference="torso">
     <selfCollide>true</selfCollide>
   </gazebo>
-  <gazebo reference="head_pan">
+  <!--gazebo reference="head_pan">
     <implicitSpringDamper>1</implicitSpringDamper>
-  </gazebo>
+  </gazebo-->
   <gazebo reference="right_s0">
     <implicitSpringDamper>1</implicitSpringDamper>
@@ -78,19 +72,4 @@
         </noise>
       </camera>
-      <plugin filename="libgazebo_ros_camera.so" name="camera_controller">
-        <alwaysOn>true</alwaysOn>
-        <updateRate>0.0</updateRate>
-        <cameraName>head_camera</cameraName>
-        <imageTopicName>image</imageTopicName>
-        <cameraInfoTopicName>camera_info</cameraInfoTopicName>
-        <frameName>head_camera</frameName>
-        <hackBaseline>0.07</hackBaseline>
-        <distortionK1>0.0</distortionK1>
-        <distortionK2>0.0</distortionK2>
-        <distortionK3>0.0</distortionK3>
-        <distortionT1>0.0</distortionT1>
-        <distortionT2>0.0</distortionT2>
-        <robotNamespace>/cameras</robotNamespace>
-      </plugin>
     </sensor>
   </gazebo>
@@ -116,19 +95,4 @@
         </noise>
       </camera>
-      <plugin filename="libgazebo_ros_camera.so" name="camera_controller">
-        <alwaysOn>true</alwaysOn>
-        <updateRate>0.0</updateRate>
-        <cameraName>right_hand_camera</cameraName>
-        <imageTopicName>image</imageTopicName>
-        <cameraInfoTopicName>camera_info</cameraInfoTopicName>
-        <frameName>right_hand_camera</frameName>
-        <hackBaseline>0.07</hackBaseline>
-        <distortionK1>0.0</distortionK1>
-        <distortionK2>0.0</distortionK2>
-        <distortionK3>0.0</distortionK3>
-        <distortionT1>0.0</distortionT1>
-        <distortionT2>0.0</distortionT2>
-        <robotNamespace>/cameras</robotNamespace>
-      </plugin>
     </sensor>
   </gazebo>
@@ -154,28 +118,8 @@
         </noise>
       </camera>
-      <plugin filename="libgazebo_ros_camera.so" name="camera_controller">
-        <alwaysOn>true</alwaysOn>
-        <updateRate>0.0</updateRate>
-        <cameraName>left_hand_camera</cameraName>
-        <imageTopicName>image</imageTopicName>
-        <cameraInfoTopicName>camera_info</cameraInfoTopicName>
-        <frameName>left_hand_camera</frameName>
-        <hackBaseline>0.07</hackBaseline>
-        <distortionK1>0.0</distortionK1>
-        <distortionK2>0.0</distortionK2>
-        <distortionK3>0.0</distortionK3>
-        <distortionT1>0.0</distortionT1>
-        <distortionT2>0.0</distortionT2>
-        <robotNamespace>/cameras</robotNamespace>
-      </plugin>
     </sensor>
   </gazebo>
   <gazebo reference="display">
     <visual>
-      <plugin name="screen_video_controller" filename="libgazebo_ros_video.so">
-        <height>600</height>
-        <width>1024</width>
-        <topicName>/robot/xdisplay</topicName>
-      </plugin>
     </visual>
   </gazebo>
@@ -203,11 +147,4 @@
         </range>
       </ray>
-      <plugin name="sonar_plugin" filename="libgazebo_ros_block_laser.so">
-        <gaussianNoise>0.00</gaussianNoise>
-        <alwaysOn>true</alwaysOn>
-        <updateRate>100.0</updateRate>
-        <topicName>/robot/sonar/head_sonar/state</topicName>
-        <frameName>sonar_ring</frameName>
-      </plugin>
       <always_on>true</always_on>
       <update_rate>100.0</update_rate>
@@ -231,11 +168,4 @@
         </range>
       </ray>
-      <plugin name="plugin_3" filename="libgazebo_ros_laser.so">
-        <gaussianNoise>0.005</gaussianNoise>
-        <alwaysOn>true</alwaysOn>
-        <updateRate>100</updateRate>
-        <topicName>/sim/laserscan/right_hand_range/state</topicName>
-        <frameName>right_hand_range</frameName>
-      </plugin>
       <always_on>true</always_on>
       <update_rate>100.0</update_rate>
@@ -259,168 +189,7 @@
         </range>
       </ray>
-      <plugin name="plugin_4" filename="libgazebo_ros_laser.so">
-        <gaussianNoise>0.005</gaussianNoise>
-        <alwaysOn>true</alwaysOn>
-        <updateRate>100</updateRate>
-        <topicName>/sim/laserscan/left_hand_range/state</topicName>
-        <frameName>left_hand_range</frameName>
-      </plugin>
       <always_on>true</always_on>
       <update_rate>100.0</update_rate>
     </sensor>
   </gazebo>
-  <!-- Transmissions -->
-  <!-- Right Arm -->
-  <transmission name="right_tran1">
-    <type>transmission_interface/SimpleTransmission</type>
-    <joint name="right_s0">
-      <hardwareInterface>EffortJointInterface</hardwareInterface>
-    </joint>
-    <actuator name="right_motor1">
-      <hardwareInterface>EffortJointInterface</hardwareInterface>
-      <mechanicalReduction>1</mechanicalReduction>
-    </actuator>
-  </transmission>
-  <transmission name="right_tran2">
-    <type>transmission_interface/SimpleTransmission</type>
-    <joint name="right_s1">
-      <hardwareInterface>EffortJointInterface</hardwareInterface>
-    </joint>
-    <actuator name="right_motor2">
-      <hardwareInterface>EffortJointInterface</hardwareInterface>
-      <mechanicalReduction>1</mechanicalReduction>
-    </actuator>
-  </transmission>
-  <transmission name="right_tran3">
-    <type>transmission_interface/SimpleTransmission</type>
-    <joint name="right_e0">
-      <hardwareInterface>EffortJointInterface</hardwareInterface>
-    </joint>
-    <actuator name="right_motor3">
-      <hardwareInterface>EffortJointInterface</hardwareInterface>
-      <mechanicalReduction>1</mechanicalReduction>
-    </actuator>
-  </transmission>
-  <transmission name="right_tran4">
-    <type>transmission_interface/SimpleTransmission</type>
-    <joint name="right_e1">
-      <hardwareInterface>EffortJointInterface</hardwareInterface>
-    </joint>
-    <actuator name="right_motor4">
-      <hardwareInterface>EffortJointInterface</hardwareInterface>
-      <mechanicalReduction>1</mechanicalReduction>
-    </actuator>
-  </transmission>
-  <transmission name="right_tran5">
-    <type>transmission_interface/SimpleTransmission</type>
-    <joint name="right_w0">
-      <hardwareInterface>EffortJointInterface</hardwareInterface>
-    </joint>
-    <actuator name="right_motor5">
-      <hardwareInterface>EffortJointInterface</hardwareInterface>
-      <mechanicalReduction>1</mechanicalReduction>
-    </actuator>
-  </transmission>
-  <transmission name="right_tran6">
-    <type>transmission_interface/SimpleTransmission</type>
-    <joint name="right_w1">
-      <hardwareInterface>EffortJointInterface</hardwareInterface>
-    </joint>
-    <actuator name="right_motor6">
-      <hardwareInterface>EffortJointInterface</hardwareInterface>
-      <mechanicalReduction>1</mechanicalReduction>
-    </actuator>
-  </transmission>
-  <transmission name="right_tran7">
-    <type>transmission_interface/SimpleTransmission</type>
-    <joint name="right_w2">
-      <hardwareInterface>EffortJointInterface</hardwareInterface>
-    </joint>
-    <actuator name="right_motor7">
-      <hardwareInterface>EffortJointInterface</hardwareInterface>
-      <mechanicalReduction>1</mechanicalReduction>
-    </actuator>
-  </transmission>
-  <!-- Left Arm -->
-  <transmission name="left_tran1">
-    <type>transmission_interface/SimpleTransmission</type>
-    <joint name="left_s0">
-      <hardwareInterface>EffortJointInterface</hardwareInterface>
-    </joint>
-    <actuator name="left_motor1">
-      <hardwareInterface>EffortJointInterface</hardwareInterface>
-      <mechanicalReduction>1</mechanicalReduction>
-    </actuator>
-  </transmission>
-  <transmission name="left_tran2">
-    <type>transmission_interface/SimpleTransmission</type>
-    <joint name="left_s1">
-      <hardwareInterface>EffortJointInterface</hardwareInterface>
-    </joint>
-    <actuator name="left_motor2">
-      <hardwareInterface>EffortJointInterface</hardwareInterface>
-      <mechanicalReduction>1</mechanicalReduction>
-    </actuator>
-  </transmission>
-  <transmission name="left_tran3">
-    <type>transmission_interface/SimpleTransmission</type>
-    <joint name="left_e0">
-      <hardwareInterface>EffortJointInterface</hardwareInterface>
-    </joint>
-    <actuator name="left_motor3">
-      <hardwareInterface>EffortJointInterface</hardwareInterface>
-      <mechanicalReduction>1</mechanicalReduction>
-    </actuator>
-  </transmission>
-  <transmission name="left_tran4">
-    <type>transmission_interface/SimpleTransmission</type>
-    <joint name="left_e1">
-      <hardwareInterface>EffortJointInterface</hardwareInterface>
-    </joint>
-    <actuator name="left_motor4">
-      <hardwareInterface>EffortJointInterface</hardwareInterface>
-      <mechanicalReduction>1</mechanicalReduction>
-    </actuator>
-  </transmission>
-  <transmission name="left_tran5">
-    <type>transmission_interface/SimpleTransmission</type>
-    <joint name="left_w0">
-      <hardwareInterface>EffortJointInterface</hardwareInterface>
-    </joint>
-    <actuator name="left_motor5">
-      <hardwareInterface>EffortJointInterface</hardwareInterface>
-      <mechanicalReduction>1</mechanicalReduction>
-    </actuator>
-  </transmission>
-  <transmission name="left_tran6">
-    <type>transmission_interface/SimpleTransmission</type>
-    <joint name="left_w1">
-      <hardwareInterface>EffortJointInterface</hardwareInterface>
-    </joint>
-    <actuator name="left_motor6">
-      <hardwareInterface>EffortJointInterface</hardwareInterface>
-      <mechanicalReduction>1</mechanicalReduction>
-    </actuator>
-  </transmission>
-  <transmission name="left_tran7">
-    <type>transmission_interface/SimpleTransmission</type>
-    <joint name="left_w2">
-      <hardwareInterface>EffortJointInterface</hardwareInterface>
-    </joint>
-    <actuator name="left_motor7">
-      <hardwareInterface>EffortJointInterface</hardwareInterface>
-      <mechanicalReduction>1</mechanicalReduction>
-    </actuator>
-  </transmission>
-  <!-- Head -->
-  <transmission name="head1">
-    <type>transmission_interface/SimpleTransmission</type>
-    <joint name="head_pan">
-      <hardwareInterface>EffortJointInterface</hardwareInterface>
-    </joint>
-    <actuator name="head_motor1">
-      <hardwareInterface>EffortJointInterface</hardwareInterface>
-      <mechanicalReduction>1</mechanicalReduction>
-    </actuator>
-  </transmission>
 </robot>

File: baxter_description/urdf/baxter_base/baxter_base.urdf.xacro (robot description, xacro)
@@ -1,5 +1,5 @@
 <?xml version="1.0" ?>
 <robot name="baxter" xmlns:xacro="http://www.ros.org/wiki/xacro">
-<!--  <xacro:if value="$(arg gazebo)">
+ <xacro:if value="$(arg gazebo)">
     <xacro:property name="mass_scale" value=".1"/>
     <xacro:include filename="$(find baxter_description)/urdf/baxter_base/baxter_base.gazebo.xacro" />
@@ -7,7 +7,7 @@
   <xacro:unless value="$(arg gazebo)">
     <xacro:property name="mass_scale" value=".1"/>
-  </xacro:unless>-->
+  </xacro:unless>
   <xacro:macro name="range_sensor" params="side">
- <!-- <gazebo>
+<gazebo>
   <sensor name="range_${side}" type="gpu_lidar">
     <pose >1 0 0 0 ${PI/2} 0</pose>
@@ -38,5 +38,5 @@
     <visualize>true</visualize>
 </sensor>
-</gazebo>-->
+</gazebo>
 </xacro:macro>
   <link name="base">
@@ -249,5 +249,5 @@
     <child link="right_torso_itb"/>
   </joint>
-  <joint name="head_pan" type="revolute">
+  <!--joint name="head_pan" type="revolute">
     <origin rpy="0 0 0" xyz="0.06 0 0.686"/>
     <axis xyz="0 0 1"/>
@@ -255,5 +255,10 @@
     <child link="head"/>
     <limit effort="50000" lower="-1.3963" upper="1.3963" velocity="10000"/>
-    <dynamics damping="0.7" friction="0.0"/>
+    <dynamics damping="10000.0" friction="100000.0"/>
+  </joint-->
+  <joint name="head_pan" type="fixed">
+    <origin rpy="0 0 0" xyz="0.06 0 0.686"/>
+    <parent link="torso"/>
+    <child link="head"/>
   </joint>
   <joint name="head_nod" type="fixed">
@@ -553,5 +558,5 @@
     <child link="right_upper_shoulder"/>
     <limit effort="50.0" lower="-1.70167993878" upper="1.70167993878" velocity="1.5"/>
-    <dynamics damping="0.7" friction="0.0"/>
+    <dynamics damping="10000.0" friction="100000.0"/>
   </joint>
   <joint name="right_s1" type="revolute">
@@ -561,5 +566,5 @@
     <child link="right_lower_shoulder"/>
     <limit effort="50.0" lower="-2.147" upper="1.047" velocity="1.5"/>
-    <dynamics damping="0.7" friction="0.0"/>
+    <dynamics damping="10000.0" friction="100000.0"/>
   </joint>
   <joint name="right_e0" type="revolute">
@@ -569,5 +574,5 @@
     <child link="right_upper_elbow"/>
     <limit effort="50.0" lower="-3.05417993878" upper="3.05417993878" velocity="1.5"/>
-    <dynamics damping="0.7" friction="0.0"/>
+    <dynamics damping="10000.0" friction="100000.0"/>
   </joint>
   <joint name="right_e0_fixed" type="fixed">
@@ -583,5 +588,5 @@
     <child link="right_lower_elbow"/>
     <limit effort="50.0" lower="-0.05" upper="2.618" velocity="1.5"/>
-    <dynamics damping="0.7" friction="0.0"/>
+    <dynamics damping="10000.0" friction="100000.0"/>
   </joint>
   <joint name="right_w0" type="revolute">
@@ -591,5 +596,5 @@
     <child link="right_upper_forearm"/>
     <limit effort="15.0" lower="-3.059" upper="3.059" velocity="4.0"/>
-    <dynamics damping="0.7" friction="0.0"/>
+    <dynamics damping="10000.0" friction="100000.0"/>
   </joint>
   <joint name="right_w0_fixed" type="fixed">
@@ -611,5 +616,5 @@
     <child link="right_lower_forearm"/>
     <limit effort="15.0" lower="-1.57079632679" upper="2.094" velocity="4.0"/>
-    <dynamics damping="0.7" friction="0.0"/>
+    <dynamics damping="10000.0" friction="100000.0"/>
   </joint>
   <joint name="right_w2" type="revolute">
@@ -619,5 +624,5 @@
     <child link="right_wrist"/>
     <limit effort="15.0" lower="-3.059" upper="3.059" velocity="4.0"/>
-    <dynamics damping="0.7" friction="0.0"/>
+    <dynamics damping="10000.0" friction="100000.0"/>
   </joint>
   <joint name="right_hand_fixed" type="fixed">
@@ -922,5 +927,5 @@
     <child link="left_upper_shoulder"/>
     <limit effort="50.0" lower="-1.70167993878" upper="1.70167993878" velocity="1.5"/>
-    <dynamics damping="0.7" friction="0.0"/>
+    <dynamics damping="10000.0" friction="100000.0"/>
   </joint>
   <joint name="left_s1" type="revolute">
@@ -930,5 +935,5 @@
     <child link="left_lower_shoulder"/>
     <limit effort="50.0" lower="-2.147" upper="1.047" velocity="1.5"/>
-    <dynamics damping="0.7" friction="0.0"/>
+    <dynamics damping="10000.0" friction="100000.0"/>
   </joint>
   <joint name="left_e0" type="revolute">
@@ -938,5 +943,5 @@
     <child link="left_upper_elbow"/>
     <limit effort="50.0" lower="-3.05417993878" upper="3.05417993878" velocity="1.5"/>
-    <dynamics damping="0.7" friction="0.0"/>
+    <dynamics damping="10000.0" friction="100000.0"/>
   </joint>
   <joint name="left_e0_fixed" type="fixed">
@@ -952,5 +957,5 @@
     <child link="left_lower_elbow"/>
     <limit effort="50.0" lower="-0.05" upper="2.618" velocity="1.5"/>
-    <dynamics damping="0.7" friction="0.0"/>
+    <dynamics damping="10000.0" friction="100000.0"/>
   </joint>
   <joint name="left_w0" type="revolute">
@@ -960,5 +965,5 @@
     <child link="left_upper_forearm"/>
     <limit effort="15.0" lower="-3.059" upper="3.059" velocity="4.0"/>
-    <dynamics damping="0.7" friction="0.0"/>
+    <dynamics damping="10000.0" friction="100000.0"/>
   </joint>
   <joint name="left_w0_fixed" type="fixed">
@@ -980,5 +985,5 @@
     <child link="left_lower_forearm"/>
     <limit effort="15.0" lower="-1.57079632679" upper="2.094" velocity="4.0"/>
-    <dynamics damping="0.7" friction="0.0"/>
+    <dynamics damping="10000.0" friction="100000.0"/>
   </joint>
   <joint name="left_w2" type="revolute">
@@ -988,5 +993,5 @@
     <child link="left_wrist"/>
     <limit effort="15.0" lower="-3.059" upper="3.059" velocity="4.0"/>
-    <dynamics damping="0.7" friction="0.0"/>
+    <dynamics damping="10000.0" friction="100000.0"/>
   </joint>
   <joint name="left_hand_fixed" type="fixed">

File: baxter_description/urdf/pedestal/pedestal.xacro (robot description, xacro)
@@ -2,5 +2,5 @@
 <robot name="pedestal" xmlns:xacro="http://www.ros.org/wiki/xacro">
   <!-- Arguments and Defaults-->
-<!--   <xacro:arg name="gazebo" default="false"/> -->
+  <xacro:arg name="gazebo" default="true"/>
   <link name="pedestal">
     <visual>
@@ -30,5 +30,5 @@
     <child link="pedestal"/>
   </joint>
-  <!--<xacro:if value="$(arg gazebo)">
+  <!--xacro:if value="$(arg gazebo)">
     <link name="world"/>
     <joint name="fixed" type="fixed">
@@ -36,4 +36,4 @@
       <child link="base"/>
     </joint>
-  </xacro:if>-->
+  </xacro:if-->
 </robot>

File: rethink_ee_description/urdf/electric_gripper/rethink_electric_gripper.xacro (robot description, xacro)
@@ -60,42 +60,22 @@
     <xacro:property name="l_finger_offset" value="${((l_finger_slot-1)*0.0095) -0.011}" scope="local"/>
     <joint name="${gripper_side}_gripper_l_finger_joint" type="prismatic">
-      <origin rpy="0 0 0" xyz="0.0 ${l_finger_offset} 0.02"/>
-      <axis xyz="0 1 0"/>
+      <origin rpy="0 0 0" xyz="0.0 0.02 0.02"/>
+      <axis xyz="0 -1 0"/>
       <parent link="${side}_gripper_base"/>
       <child link="${gripper_side}_gripper_l_finger"/>
       <limit effort="20.0" lower="0.0" upper="0.020833" velocity="5.0"/>
-      <dynamics damping="0.7" friction="0.0"/>
+      <dynamics damping="100.0" friction="100.0"/>
     </joint>
     <!-- Right finger -->
     <xacro:property name="r_finger_offset" value="${((r_finger_slot-1)*-0.0095) +0.011}" scope="local"/>
     <joint name="${gripper_side}_gripper_r_finger_joint" type="prismatic">
-      <origin rpy="0 0 0" xyz="0.0 ${r_finger_offset} 0.02"/>
-      <axis xyz="0 1 0"/>
+      <origin rpy="0 0 0" xyz="0.0 -0.02 0.02"/>
+      <axis xyz="0 -1 0"/>
       <parent link="${side}_gripper_base"/>
       <child link="${gripper_side}_gripper_r_finger"/>
       <limit effort="20.0" lower="-0.020833" upper="0.0" velocity="5.0"/>
-      <mimic joint="${gripper_side}_gripper_l_finger_joint" multiplier="-1.0"/>
-      <dynamics damping="0.7" friction="0.0"/>
+      <!--mimic joint="${gripper_side}_gripper_l_finger_joint" multiplier="-1.0"/-->
+      <dynamics damping="100.0" friction="100.0"/>
     </joint>
-    <transmission name="gripper_${side}1">
-      <type>transmission_interface/SimpleTransmission</type>
-      <joint name="${gripper_side}_gripper_r_finger_joint">
-        <hardwareInterface>EffortJointInterface</hardwareInterface>
-      </joint>
-      <actuator name="gripper_${gripper_side}1_motor1">
-        <hardwareInterface>EffortJointInterface</hardwareInterface>
-        <mechanicalReduction>1</mechanicalReduction>
-      </actuator>
-    </transmission>
-    <transmission name="gripper_${side}2">
-      <type>transmission_interface/SimpleTransmission</type>
-      <joint name="${gripper_side}_gripper_l_finger_joint">
-        <hardwareInterface>EffortJointInterface</hardwareInterface>
-      </joint>
-      <actuator name="gripper_${gripper_side}1_motor2">
-        <hardwareInterface>EffortJointInterface</hardwareInterface>
-        <mechanicalReduction>1</mechanicalReduction>
-      </actuator>
-    </transmission>
     <gazebo reference="${gripper_side}_gripper_r_finger_joint">
       <implicitSpringDamper>1</implicitSpringDamper>
